File: rf-rfid/prj-kicad/pmod-rfid.kicad_pcb (KiCad board)
At the start: 2 copper layers, 38.1 x 20.3 mm, 34 parts, among them P1 PMOD, P2 ANTENNA, U1 TRF7970, X1 13,56MHz

Commit message: rf_rfid updated
Parts:
- removed R2, R3: 0, pmod-rfid:SMD0402
- removed agilack-11.5: 450px, pmod-rfid:logo-agilack-11.5
- removed ohw_logo: VAL**, pmod-rfid:logo-ohw
Connections:
- R1 pad 1: GND -> +Vrfid
- U1 pad 17: SPI_CFG0 -> Net-(U1-Pad17)
- U1 pad 18: SPI_CFG1 -> +Vrfid
- U1 pad 19: SPI_CFG1 -> +Vrfid
Routing:
- net +Vrfid: track 55.1 -> 68.8 mm
- net SPI_CFG1: track 2.39 -> 0.00 mm
- net GND: track 171.1 -> 169.6 mm
- net SPI_SCK: track 16.7 -> 17.9 mm
- net SPI_CFG0: track 1.15 -> 0.00 mm
- net Net-(U1-Pad17): track 0.00 -> 1.15 mm

Commit message: rf-rfid finished
Connections:
- U1 pad 17: Net-(U1-Pad17) -> GND
Routing:
- net GND: track 169.6 -> 171.1 mm
- net +Vrfid: track 68.8 -> 67.4 mm
- net Net-(U1-Pad17): track 1.15 -> 0.00 mm
Changed lines of the file:
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@@
     (thickness 1.6)
     (drawings 8)
-    (tracks 340)
+    (tracks 332)
     (zones 0)
     (modules 30)
-    (nets 31)
+    (nets 30)
   )
   (page A4)
@@
   )
   (setup
-    (last_trace_width 0.2032)
+    (last_trace_width 0.25)
     (user_trace_width 0.2032)
     (user_trace_width 0.3048)
@@
   (net 28 +3.3V)
   (net 29 RESET)
-  (net 30 "Net-(U1-Pad17)")
   (net_class Default "This is the default net class."
     (clearance 0.1524)
@@
     (add_net "Net-(TP1-Pad1)")
     (add_net "Net-(TP2-Pad1)")
-    (add_net "Net-(U1-Pad17)")
     (add_net "Net-(U1-Pad20)")
     (add_net "Net-(U1-Pad22)")
@@
       (net 12 +Vrfid))
     (pad 17 smd rect (at 1.75006 -2.49936) (size 0.2794 0.8509) (layers F.Cu F.Paste F.Mask)
-      (net 30 "Net-(U1-Pad17)"))
+      (net 27 GND))
     (pad 25 smd rect (at -2.49936 -1.75006 90) (size 0.2794 0.8509) (layers F.Cu F.Paste F.Mask)
       (net 27 GND))
@@
   (segment (start 150.25006 103.42516) (end 151.3078 104.4829) (width 0.2032) (layer F.Cu) (net 4))
   (segment (start 151.8539 108.6485) (end 153.4287 108.6485) (width 0.4064) (layer F.Cu) (net 4))
-  (segment (start 150.25006 97.50064) (end 150.25006 96.56682) (width 0.2032) (layer F.Cu) (net 30))
-  (segment (start 150.25006 96.56682) (end 150.4061 96.41078) (width 0.2032) (layer F.Cu) (net 30))
   (segment (start 153.4287 105.4608) (end 155.3444 105.4608) (width 0.2032) (layer F.Cu) (net 5))
   (segment (start 155.3444 105.4608) (end 155.7274 105.0778) (width 0.2032) (layer F.Cu) (net 5))
@@
   (via (at 151.1173 97.3836) (size 0.7112) (drill 0.3048) (layers F.Cu B.Cu) (net 12))
   (segment (start 151.1189 97.382) (end 151.1173 97.3836) (width 0.25) (layer F.Cu) (net 12))
-  (segment (start 148.68838 95.51162) (end 148.52 95.68) (width 0.2032) (layer F.Cu) (net 12))
-  (segment (start 148.68838 95.51162) (end 149.3901 95.51162) (width 0.2032) (layer F.Cu) (net 12))
   (via (at 148.52 96.14) (size 0.7112) (drill 0.3048) (layers F.Cu B.Cu) (net 12))
-  (segment (start 148.52 95.68) (end 148.52 96.14) (width 0.2032) (layer F.Cu) (net 12))
-  (segment (start 149.37848 95.5) (end 149.3901 95.51162) (width 0.3048) (layer F.Cu) (net 12))
-  (segment (start 149.37848 95.5) (end 149.3901 95.51162) (width 0.2032) (layer F.Cu) (net 12))
   (segment (start 140.7414 106.5022) (end 140.7414 105.8164) (width 0.3048) (layer F.Cu) (net 12))
   (segment (start 140.7414 105.8164) (end 141.3637 105.1941) (width 0.3048) (layer F.Cu) (net 12))
@@
   (via (at 151.2697 95.5167) (size 0.7112) (drill 0.3048) (layers F.Cu B.Cu) (net 27))
   (segment (start 152.41 95.858) (end 151.611 95.858) (width 0.2032) (layer F.Cu) (net 27))
-  (segment (start 150.92172 95.51162) (end 150.9268 95.5167) (width 0.2032) (layer F.Cu) (net 27))
-  (segment (start 150.9268 95.5167) (end 151.2697 95.5167) (width 0.2032) (layer F.Cu) (net 27))
-  (segment (start 150.92172 95.51162) (end 150.4061 95.51162) (width 0.2032) (layer F.Cu) (net 27))
   (segment (start 151.611 95.858) (end 151.2697 95.5167) (width 0.2032) (layer F.Cu) (net 27))
   (segment (start 146.2913 106.8578) (end 146.2913 108.9152) (width 0.3048) (layer B.Cu) (net 27))
@@
   (via (at 152.2222 98.7425) (size 0.7112) (drill 0.3048) (layers F.Cu B.Cu) (net 27))
   (segment (start 150.99936 98.75032) (end 149.74968 98.75032) (width 0.2032) (layer F.Cu) (net 27))
+  (segment (start 150.25006 96.53634) (end 150.25006 97.50064) (width 0.25) (layer F.Cu) (net 27))
+  (segment (start 151.2697 95.5167) (end 150.25006 96.53634) (width 0.25) (layer F.Cu) (net 27))
   (segment (start 140.7414 108.0262) (end 140.7414 110.1586) (width 0.3048) (layer F.Cu) (net 28))
   (segment (start 139.8705 111.0295) (end 138.8137 111.0295) (width 0.3048) (layer F.Cu) (net 28))
