File: rf-rfid/prj-kicad/pmod-rfid.sch (KiCad schematic (older format))
At the start: 33 parts, among them P1 PMOD, P2 ANTENNA, U1 TRF7970, X1 13,56MHz

Commit message: rf_rfid updated
Parts:
- removed C17: CP, symbol CP
- removed R2, R3: 0, pmod-rfid:SMD0402, symbol R
- C1, C10, C11, C12, C13, C14, C15, C16, C18, C19, C2, C20, C3, C4, C5, C6, C7, C8, C9: symbol C -> pmod-rfid:C
- L1, L2, L3: symbol INDUCTOR -> pmod-rfid:INDUCTOR
- P1: symbol PMOD -> pmod-rfid:PMOD
- P2: symbol ANTENNA -> pmod-rfid:ANTENNA
- R1: symbol R -> pmod-rfid:R
- TP1, TP2, TP3: symbol CONN_1 -> pmod-rfid:CONN_1
- U1: symbol TRF7970 -> pmod-rfid:TRF7970
- X1: symbol CRYSTAL4 -> pmod-rfid:CRYSTAL4
Connections:
- net labels removed: SPI_CFG0, SPI_CFG1, SPI_CFG2
- wire segments 124 -> 137

Commit message: rf-rfid finished
Connections:
- net GND: now also U1.17 (IO0)
Changed lines of the file:
@@
 Wire Wire Line
 	5300 3150 5300 3100
-$Comp
-L pmod-rfid:GND #PWR023
-U 1 1 5A342BF8
-P 6330 4400
-F 0 "#PWR023" H 6330 4400 30  0001 C CNN
-F 1 "GND" H 6330 4330 30  0001 C CNN
-F 2 "" H 6330 4400 60  0000 C CNN
-F 3 "" H 6330 4400 60  0000 C CNN
-	1    6330 4400
-	-1   0    0    -1
-$EndComp
 NoConn ~ 6100 4800
 NoConn ~ 6100 5100
@@
 	6100 4650 6725 4650
 Wire Wire Line
-	6325 4400 6325 4350
-Wire Wire Line
-	6100 4350 6325 4350
+	6100 4350 6370 4350
+Wire Wire Line
+	6370 4350 6370 4420
+$Comp
+L pmod-rfid:GND #PWR?
+U 1 1 5C7C5405
+P 6370 4420
+F 0 "#PWR?" H 6370 4420 30  0001 C CNN
+F 1 "GND" H 6370 4350 30  0001 C CNN
+F 2 "" H 6370 4420 60  0000 C CNN
+F 3 "" H 6370 4420 60  0000 C CNN
+	1    6370 4420
+	1    0    0    -1
+$EndComp
 $EndSCHEMATC
